Commit message: Added hokuyo sensor

File: urdf/lidar.xacro (robot description, xacro)
@@ -24,5 +24,5 @@
     <gazebo reference="laser_frame">
         <material>Gazebo/Red</material>
-        <sensor name="laser" type="ray">
+        <sensor name="lidar" type="ray">
             <pose> 0 0 0 0 0 0 </pose>
             <visualize>true</visualize>
@@ -41,7 +41,7 @@
                 </range>
             </ray>
-            <plugin name="laser_controller" filename="libgazebo_ros_ray_sensor.so">
+            <plugin name="scan" filename="libgazebo_ros_ray_sensor.so">
                 <ros>
-                    <argument>~/out:=scan</argument>
+                    <remapping>scan</remapping>
                 </ros>
                 <output_type>sensor_msgs/LaserScan</output_type>

File: urdf/rupert.xacro (robot description, xacro)
@@ -41,5 +41,5 @@
   <xacro:include filename="$(find rupert_learns)/urdf/materials.xacro" />
    <xacro:include filename="inertial_macros.xacro"/>
-  <xacro:include filename="$(find rupert_learns)/urdf/lidar.xacro" />
+  <!-- <xacro:include filename="$(find rupert_learns)/urdf/lidar.xacro" /> -->
   <!-- Used for fixing robot to Gazebo 'base_link' -->
 <link name = "dummy"/>
@@ -71,4 +71,25 @@
     </inertial>
   </link>
+  <joint name="laser_joint" type="fixed">
+      <parent link="body"/>
+      <child link="hokuyo_link"/>
+      <origin xyz="0.1 0 0.175" rpy="0 0 0"/>
+  </joint>
+  <link name="hokuyo_link">
+      <visual>
+          <geometry>
+              <cylinder radius="0.05" length="0.04"/>
+          </geometry>
+          <material name="red"/>
+      </visual>
+      <collision>
+          <geometry>
+              <cylinder radius="0.05" length="0.04"/>
+          </geometry>
+      </collision>
+      <xacro:inertial_cylinder mass="0.1" length="0.04" radius="0.05">
+          <origin xyz="0 0 0" rpy="0 0 0"/>
+      </xacro:inertial_cylinder>
+    </link>
   <link name="block1">
     <collision>
