Commit message: Created damaged robot

File: urdf/rupert.xacro (robot description, xacro)
@@ -69,5 +69,5 @@
     </inertial>
   </link>
-  <link name="block1">
+  <!-- <link name="block1">
     <collision>
       <origin xyz="0 0 0" rpy="0 0 0"/>
@@ -91,5 +91,5 @@
     izz="${mass_block / 12.0 * (block_width*block_width + block_length*block_length)}"/>
     </inertial>
-  </link>
+  </link> -->
     <link name="block2">
     <collision>
@@ -161,10 +161,10 @@
     </inertial>
   </link>
-  <joint name="block_j1" type="fixed">
+  <!-- <joint name="block_j1" type="fixed">
     <parent link="body"/>
     <child link="block1"/>
     <origin xyz="${body_width/2} ${body_length/2} 0" rpy="0 0 0.785398"/>
     <axis xyz="0 0 1" />
-  </joint>
+  </joint> -->
   <joint name="block_j2" type="fixed">
     <parent link="body"/>
@@ -185,5 +185,5 @@
     <axis xyz="0 0 1" />
   </joint>
-  <joint name="hip_j1" type="revolute">
+  <!-- <joint name="hip_j1" type="revolute">
     <parent link="block1"/>
     <child link="hip1"/>
@@ -191,5 +191,5 @@
     <axis xyz="0 0 1" />
     <limit effort="300" velocity="1.0" lower="-1.7" upper="1.7"/>
-  </joint>
+  </joint> -->
     <joint name="hip_j2" type="revolute">
     <parent link="block2"/>
@@ -214,5 +214,5 @@
   </joint>
   <!-- Base Link -->
-  <link name="hip1">
+  <!-- <link name="hip1">
     <collision>
       <origin xyz="${-hip_width/2} 0 0" rpy="0 0 0"/>
@@ -236,5 +236,5 @@
 	  izz="${mass_hip / 12.0 * (hip_length*hip_length + hip_width*hip_width)}"/>
     </inertial>
-  </link>
+  </link> -->
     <link name="hip2">
     <collision>
@@ -306,5 +306,5 @@
     </inertial>
   </link>
-  <joint name="knee_j1" type="revolute">
+  <!-- <joint name="knee_j1" type="revolute">
     <parent link="hip1"/>
     <child link="leg1"/>
@@ -313,5 +313,5 @@
     <dynamics damping="0.7"/>
     <limit effort="300" velocity="1.0" lower="-1.7" upper="1.7"/>
-  </joint>
+  </joint> -->
   <joint name="knee_j2" type="revolute">
     <parent link="hip2"/>
@@ -339,5 +339,5 @@
   </joint>
   <!-- Middle Link -->
-  <link name="leg1">
+  <!-- <link name="leg1">
     <collision>
       <origin xyz="0 0 ${leg_height/2}" rpy="0 0 0"/>
@@ -361,5 +361,5 @@
 	  izz="${mass_leg / 12.0 * (leg_width*leg_width + leg_length*leg_length)}"/>
     </inertial>
-  </link>
+  </link> -->
     <link name="leg2">
     <collision>
@@ -431,5 +431,5 @@
     </inertial>
   </link>
-  <joint name="ankle_j1" type="revolute">
+  <!-- <joint name="ankle_j1" type="revolute">
     <parent link="leg1"/>
     <child link="foot1"/>
@@ -438,5 +438,5 @@
     <dynamics damping="0.7"/>
     <limit effort="300" velocity="1.0" lower="-1.7" upper="1.7"/>
-  </joint>
+  </joint> -->
   <joint name="ankle_j2" type="revolute">
     <parent link="leg2"/>
@@ -464,5 +464,5 @@
   </joint>
   <!-- Top Link -->
-  <link name="foot1">
+  <!-- <link name="foot1">
     <collision>
       <origin xyz="0 0 ${foot_height/2}" rpy="0 0 0"/>
@@ -486,5 +486,5 @@
 	  izz="${mass_foot / 12.0 * (foot_width*foot_width + foot_length*foot_length)}"/>
     </inertial>
-  </link>
+  </link> -->
     <link name="foot2">
     <collision>
@@ -556,5 +556,5 @@
     </inertial>
   </link>
-  <transmission name="tran1">
+  <!-- <transmission name="tran1">
     <type>transmission_interface/SimpleTransmission</type>
     <joint name="hip_j1">
@@ -565,5 +565,5 @@
       <mechanicalReduction>1</mechanicalReduction>
     </actuator>
-  </transmission>
+  </transmission> -->
   <transmission name="tran2">
     <type>transmission_interface/SimpleTransmission</type>
@@ -596,5 +596,5 @@
     </actuator>
   </transmission>
-  <transmission name="tran5">
+  <!-- <transmission name="tran5">
     <type>transmission_interface/SimpleTransmission</type>
     <joint name="knee_j1">
@@ -605,5 +605,5 @@
       <mechanicalReduction>1</mechanicalReduction>
     </actuator>
-  </transmission>
+  </transmission> -->
   <transmission name="tran6">
     <type>transmission_interface/SimpleTransmission</type>
@@ -636,5 +636,5 @@
     </actuator>
   </transmission>
-  <transmission name="tran9">
+  <!-- <transmission name="tran9">
     <type>transmission_interface/SimpleTransmission</type>
     <joint name="ankle_j1">
@@ -645,5 +645,5 @@
       <mechanicalReduction>1</mechanicalReduction>
     </actuator>
-  </transmission>
+  </transmission> -->
   <transmission name="tran10">
     <type>transmission_interface/SimpleTransmission</type>

Commit message: Removed ankle 3

File: urdf/rupert.xacro (robot description, xacro)
@@ -69,5 +69,5 @@
     </inertial>
   </link>
-  <!-- <link name="block1">
+  <link name="block1">
     <collision>
       <origin xyz="0 0 0" rpy="0 0 0"/>
@@ -91,5 +91,5 @@
     izz="${mass_block / 12.0 * (block_width*block_width + block_length*block_length)}"/>
     </inertial>
-  </link> -->
+  </link>
     <link name="block2">
     <collision>
@@ -161,10 +161,10 @@
     </inertial>
   </link>
-  <!-- <joint name="block_j1" type="fixed">
+  <joint name="block_j1" type="fixed">
     <parent link="body"/>
     <child link="block1"/>
     <origin xyz="${body_width/2} ${body_length/2} 0" rpy="0 0 0.785398"/>
     <axis xyz="0 0 1" />
-  </joint> -->
+  </joint>
   <joint name="block_j2" type="fixed">
     <parent link="body"/>
@@ -185,5 +185,5 @@
     <axis xyz="0 0 1" />
   </joint>
-  <!-- <joint name="hip_j1" type="revolute">
+  <joint name="hip_j1" type="revolute">
     <parent link="block1"/>
     <child link="hip1"/>
@@ -191,5 +191,5 @@
     <axis xyz="0 0 1" />
     <limit effort="300" velocity="1.0" lower="-1.7" upper="1.7"/>
-  </joint> -->
+  </joint>
     <joint name="hip_j2" type="revolute">
     <parent link="block2"/>
@@ -214,5 +214,5 @@
   </joint>
   <!-- Base Link -->
-  <!-- <link name="hip1">
+  <link name="hip1">
     <collision>
       <origin xyz="${-hip_width/2} 0 0" rpy="0 0 0"/>
@@ -236,5 +236,5 @@
 	  izz="${mass_hip / 12.0 * (hip_length*hip_length + hip_width*hip_width)}"/>
     </inertial>
-  </link> -->
+  </link>
     <link name="hip2">
     <collision>
@@ -306,5 +306,5 @@
     </inertial>
   </link>
-  <!-- <joint name="knee_j1" type="revolute">
+  <joint name="knee_j1" type="revolute">
     <parent link="hip1"/>
     <child link="leg1"/>
@@ -313,5 +313,5 @@
     <dynamics damping="0.7"/>
     <limit effort="300" velocity="1.0" lower="-1.7" upper="1.7"/>
-  </joint> -->
+  </joint>
   <joint name="knee_j2" type="revolute">
     <parent link="hip2"/>
@@ -339,5 +339,5 @@
   </joint>
   <!-- Middle Link -->
-  <!-- <link name="leg1">
+  <link name="leg1">
     <collision>
       <origin xyz="0 0 ${leg_height/2}" rpy="0 0 0"/>
@@ -361,5 +361,5 @@
 	  izz="${mass_leg / 12.0 * (leg_width*leg_width + leg_length*leg_length)}"/>
     </inertial>
-  </link> -->
+  </link>
     <link name="leg2">
     <collision>
@@ -431,5 +431,5 @@
     </inertial>
   </link>
-  <!-- <joint name="ankle_j1" type="revolute">
+  <joint name="ankle_j1" type="revolute">
     <parent link="leg1"/>
     <child link="foot1"/>
@@ -438,5 +438,5 @@
     <dynamics damping="0.7"/>
     <limit effort="300" velocity="1.0" lower="-1.7" upper="1.7"/>
-  </joint> -->
+  </joint>
   <joint name="ankle_j2" type="revolute">
     <parent link="leg2"/>
@@ -447,5 +447,5 @@
     <limit effort="300" velocity="1.0" lower="-1.7" upper="1.7"/>
   </joint>
-  <joint name="ankle_j3" type="revolute">
+  <!-- <joint name="ankle_j3" type="revolute">
     <parent link="leg3"/>
     <child link="foot3"/>
@@ -454,5 +454,5 @@
     <dynamics damping="0.7"/>
     <limit effort="300" velocity="1.0" lower="-1.7" upper="1.7"/>
-  </joint>
+  </joint> -->
   <joint name="ankle_j4" type="revolute">
     <parent link="leg4"/>
@@ -464,5 +464,5 @@
   </joint>
   <!-- Top Link -->
-  <!-- <link name="foot1">
+  <link name="foot1">
     <collision>
       <origin xyz="0 0 ${foot_height/2}" rpy="0 0 0"/>
@@ -486,5 +486,5 @@
 	  izz="${mass_foot / 12.0 * (foot_width*foot_width + foot_length*foot_length)}"/>
     </inertial>
-  </link> -->
+  </link>
     <link name="foot2">
     <collision>
@@ -510,5 +510,5 @@
     </inertial>
   </link>
-    <link name="foot3">
+    <!-- <link name="foot3">
     <collision>
       <origin xyz="0 0 ${foot_height/2}" rpy="0 0 0"/>
@@ -532,5 +532,5 @@
     izz="${mass_foot / 12.0 * (foot_width*foot_width + foot_length*foot_length)}"/>
     </inertial>
-  </link>
+  </link> -->
     <link name="foot4">
     <collision>
@@ -556,5 +556,5 @@
     </inertial>
   </link>
-  <!-- <transmission name="tran1">
+  <transmission name="tran1">
     <type>transmission_interface/SimpleTransmission</type>
     <joint name="hip_j1">
@@ -565,105 +565,105 @@
       <mechanicalReduction>1</mechanicalReduction>
     </actuator>
+  </transmission>
+  <transmission name="tran2">
+    <type>transmission_interface/SimpleTransmission</type>
+    <joint name="hip_j2">
+      <hardwareInterface>hardware_interface/EffortJointInterface</hardwareInterface>
+    </joint>
+    <actuator name="motor2">
+      <hardwareInterface>hardware_interface/EffortJointInterface</hardwareInterface>
+      <mechanicalReduction>1</mechanicalReduction>
+    </actuator>
+  </transmission>
+  <transmission name="tran3">
+    <type>transmission_interface/SimpleTransmission</type>
+    <joint name="hip_j3">
+      <hardwareInterface>hardware_interface/EffortJointInterface</hardwareInterface>
+    </joint>
+    <actuator name="motor3">
+      <hardwareInterface>hardware_interface/EffortJointInterface</hardwareInterface>
+      <mechanicalReduction>1</mechanicalReduction>
+    </actuator>
+  </transmission>
+  <transmission name="tran4">
+    <type>transmission_interface/SimpleTransmission</type>
+    <joint name="hip_j4">
+      <hardwareInterface>hardware_interface/EffortJointInterface</hardwareInterface>
+    </joint>
+    <actuator name="motor4">
+      <hardwareInterface>hardware_interface/EffortJointInterface</hardwareInterface>
+      <mechanicalReduction>1</mechanicalReduction>
+    </actuator>
+  </transmission>
+  <transmission name="tran5">
+    <type>transmission_interface/SimpleTransmission</type>
+    <joint name="knee_j1">
+      <hardwareInterface>hardware_interface/EffortJointInterface</hardwareInterface>
+    </joint>
+    <actuator name="motor5">
+      <hardwareInterface>hardware_interface/EffortJointInterface</hardwareInterface>
+      <mechanicalReduction>1</mechanicalReduction>
+    </actuator>
+  </transmission>
+  <transmission name="tran6">
+    <type>transmission_interface/SimpleTransmission</type>
+    <joint name="knee_j2">
+      <hardwareInterface>hardware_interface/EffortJointInterface</hardwareInterface>
+    </joint>
+    <actuator name="motor6">
+      <hardwareInterface>hardware_interface/EffortJointInterface</hardwareInterface>
+      <mechanicalReduction>1</mechanicalReduction>
+    </actuator>
+  </transmission>
+  <transmission name="tran7">
+    <type>transmission_interface/SimpleTransmission</type>
+    <joint name="knee_j3">
+      <hardwareInterface>hardware_interface/EffortJointInterface</hardwareInterface>
+    </joint>
+    <actuator name="motor7">
+      <hardwareInterface>hardware_interface/EffortJointInterface</hardwareInterface>
+      <mechanicalReduction>1</mechanicalReduction>
+    </actuator>
+  </transmission>
+  <transmission name="tran8">
+    <type>transmission_interface/SimpleTransmission</type>
+    <joint name="knee_j4">
+      <hardwareInterface>hardware_interface/EffortJointInterface</hardwareInterface>
+    </joint>
+    <actuator name="motor8">
+      <hardwareInterface>hardware_interface/EffortJointInterface</hardwareInterface>
+      <mechanicalReduction>1</mechanicalReduction>
+    </actuator>
+  </transmission>
+  <transmission name="tran9">
+    <type>transmission_interface/SimpleTransmission</type>
+    <joint name="ankle_j1">
+      <hardwareInterface>hardware_interface/EffortJointInterface</hardwareInterface>
+    </joint>
+    <actuator name="motor9">
+      <hardwareInterface>hardware_interface/EffortJointInterface</hardwareInterface>
+      <mechanicalReduction>1</mechanicalReduction>
+    </actuator>
+  </transmission>
+  <transmission name="tran10">
+    <type>transmission_interface/SimpleTransmission</type>
+    <joint name="ankle_j2">
+      <hardwareInterface>hardware_interface/EffortJointInterface</hardwareInterface>
+    </joint>
+    <actuator name="motor10">
+      <hardwareInterface>hardware_interface/EffortJointInterface</hardwareInterface>
+      <mechanicalReduction>1</mechanicalReduction>
+    </actuator>
+  </transmission>
+  <!-- <transmission name="tran11">
+    <type>transmission_interface/SimpleTransmission</type>
+    <joint name="ankle_j3">
+      <hardwareInterface>hardware_interface/EffortJointInterface</hardwareInterface>
+    </joint>
+    <actuator name="motor11">
+      <hardwareInterface>hardware_interface/EffortJointInterface</hardwareInterface>
+      <mechanicalReduction>1</mechanicalReduction>
+    </actuator>
   </transmission> -->
-  <transmission name="tran2">
-    <type>transmission_interface/SimpleTransmission</type>
-    <joint name="hip_j2">
-      <hardwareInterface>hardware_interface/EffortJointInterface</hardwareInterface>
-    </joint>
-    <actuator name="motor2">
-      <hardwareInterface>hardware_interface/EffortJointInterface</hardwareInterface>
-      <mechanicalReduction>1</mechanicalReduction>
-    </actuator>
-  </transmission>
-  <transmission name="tran3">
-    <type>transmission_interface/SimpleTransmission</type>
-    <joint name="hip_j3">
-      <hardwareInterface>hardware_interface/EffortJointInterface</hardwareInterface>
-    </joint>
-    <actuator name="motor3">
-      <hardwareInterface>hardware_interface/EffortJointInterface</hardwareInterface>
-      <mechanicalReduction>1</mechanicalReduction>
-    </actuator>
-  </transmission>
-  <transmission name="tran4">
-    <type>transmission_interface/SimpleTransmission</type>
-    <joint name="hip_j4">
-      <hardwareInterface>hardware_interface/EffortJointInterface</hardwareInterface>
-    </joint>
-    <actuator name="motor4">
-      <hardwareInterface>hardware_interface/EffortJointInterface</hardwareInterface>
-      <mechanicalReduction>1</mechanicalReduction>
-    </actuator>
-  </transmission>
-  <!-- <transmission name="tran5">
-    <type>transmission_interface/SimpleTransmission</type>
-    <joint name="knee_j1">
-      <hardwareInterface>hardware_interface/EffortJointInterface</hardwareInterface>
-    </joint>
-    <actuator name="motor5">
-      <hardwareInterface>hardware_interface/EffortJointInterface</hardwareInterface>
-      <mechanicalReduction>1</mechanicalReduction>
-    </actuator>
-  </transmission> -->
-  <transmission name="tran6">
-    <type>transmission_interface/SimpleTransmission</type>
-    <joint name="knee_j2">
-      <hardwareInterface>hardware_interface/EffortJointInterface</hardwareInterface>
-    </joint>
-    <actuator name="motor6">
-      <hardwareInterface>hardware_interface/EffortJointInterface</hardwareInterface>
-      <mechanicalReduction>1</mechanicalReduction>
-    </actuator>
-  </transmission>
-  <transmission name="tran7">
-    <type>transmission_interface/SimpleTransmission</type>
-    <joint name="knee_j3">
-      <hardwareInterface>hardware_interface/EffortJointInterface</hardwareInterface>
-    </joint>
-    <actuator name="motor7">
-      <hardwareInterface>hardware_interface/EffortJointInterface</hardwareInterface>
-      <mechanicalReduction>1</mechanicalReduction>
-    </actuator>
-  </transmission>
-  <transmission name="tran8">
-    <type>transmission_interface/SimpleTransmission</type>
-    <joint name="knee_j4">
-      <hardwareInterface>hardware_interface/EffortJointInterface</hardwareInterface>
-    </joint>
-    <actuator name="motor8">
-      <hardwareInterface>hardware_interface/EffortJointInterface</hardwareInterface>
-      <mechanicalReduction>1</mechanicalReduction>
-    </actuator>
-  </transmission>
-  <!-- <transmission name="tran9">
-    <type>transmission_interface/SimpleTransmission</type>
-    <joint name="ankle_j1">
-      <hardwareInterface>hardware_interface/EffortJointInterface</hardwareInterface>
-    </joint>
-    <actuator name="motor9">
-      <hardwareInterface>hardware_interface/EffortJointInterface</hardwareInterface>
-      <mechanicalReduction>1</mechanicalReduction>
-    </actuator>
-  </transmission> -->
-  <transmission name="tran10">
-    <type>transmission_interface/SimpleTransmission</type>
-    <joint name="ankle_j2">
-      <hardwareInterface>hardware_interface/EffortJointInterface</hardwareInterface>
-    </joint>
-    <actuator name="motor10">
-      <hardwareInterface>hardware_interface/EffortJointInterface</hardwareInterface>
-      <mechanicalReduction>1</mechanicalReduction>
-    </actuator>
-  </transmission>
-  <transmission name="tran11">
-    <type>transmission_interface/SimpleTransmission</type>
-    <joint name="ankle_j3">
-      <hardwareInterface>hardware_interface/EffortJointInterface</hardwareInterface>
-    </joint>
-    <actuator name="motor11">
-      <hardwareInterface>hardware_interface/EffortJointInterface</hardwareInterface>
-      <mechanicalReduction>1</mechanicalReduction>
-    </actuator>
-  </transmission>
   <transmission name="tran12">
     <type>transmission_interface/SimpleTransmission</type>
